File: sinket/sinket.brd (EAGLE design)
At the start: 36 x 36 mm, 26 parts, among them IC1 ATTINY85-20PU, IC2 TS2940CP50S

Commit message: change capacity package
the former one was probably unrealstic for the desired value
Parts:
- C2: device rcl:C025-030X050 -> rcl:C050-025X075
- moved C2 1.27 mm to (5.71, 25.7)
Changed lines of the file:
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@@
 <attribute name="REICHELT" value="TS 2940 CP50" x="19.685" y="31.75" size="1.778" layer="28" rot="MR90" display="off"/>
 </element>
-<element name="C2" library="rcl" package="C025-030X050" value="470n" x="6.985" y="25.7175" rot="R180"/>
+<element name="C2" library="rcl" package="C050-025X075" value="470n" x="5.715" y="25.7175" rot="R180"/>
 <element name="C3" library="rcl" package="E2,5-6" value="47u" x="12.3825" y="32.0675" rot="R270"/>
 <element name="F1" library="n39" package="LP60-050" value="500mA" x="5.08" y="9.8425" rot="MR180"/>
