File: sinket/sinket.sch (EAGLE design)
At the start: 22 parts, among them IC1 ATTINY85-20PU, IC2 TS2940CP50S

Commit message: change capacity package
the former one was probably unrealstic for the desired value
Parts:
- C2: device rcl:C-EU025-030X050 -> rcl:C-EU050-025X075
Changed lines of the file:
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@@
 <part name="D3" library="diode" deviceset="1N581*" device="" technology="7-B" value="1N5817-B"/>
 <part name="IC2" library="n39" deviceset="TS2940" device="S" technology="CP50"/>
-<part name="C2" library="rcl" deviceset="C-EU" device="025-030X050" value="470n"/>
+<part name="C2" library="rcl" deviceset="C-EU" device="050-025X075" value="470n"/>
 <part name="C3" library="rcl" deviceset="CPOL-EU" device="E2.5-6" value="47u"/>
 <part name="GND9" library="supply1" deviceset="GND" device=""/>
